File: mbhp_ainser64_v1.sch (EAGLE design)
At the start: 20 parts, among them IC1 MCP3208-CI/P, IC10 4051N, IC11 4051N, IC2 74HC595N, IC9 4051N, J11 1, J12 1, J13 1, J2 1

Commit message: design ready
Parts:
- removed J11, J12, J13: 1, con-lstb:MA05-2
- added JP1, JP2, JP3: M10", SparkFun-Connectors:M10"
Connections:
- net GND: now also JP1.10, JP2.10, JP3.10; no longer J11.10, J12.10, J13.10
- net N$10: now also IC10.X1, JP2.7; no longer IC11.X5, J13.1
- net N$11: now also IC10.X2, JP2.8; no longer IC11.X6, J13.3
- net N$12: now also IC10.X3, JP2.5; no longer IC11.X4, J13.4
- net N$13: now also IC10.X5, JP2.4; no longer IC11.X3, J13.8
- net N$14: now also IC10.X7, JP2.3; no longer IC11.X2, J13.5
- net N$15: now also IC10.X6, JP2.2; no longer IC11.X1, J13.6
- net N$16: now also IC10.X4, JP2.1; no longer IC11.X0, J13.7
- net N$17: now also IC11.X2, JP3.8; no longer IC10.X7, J12.2
- net N$18: now also IC11.X1, JP3.7; no longer IC10.X5, J12.1
- net N$19: now also IC11.X0, JP3.6; no longer IC10.X6, J12.3
- net N$20: now also IC11.X3, JP3.5; no longer IC10.X4, J12.4
- net N$21: now also IC11.X5, JP3.4; no longer IC10.X3, J12.8
- net N$22: now also IC11.X7, JP3.3; no longer IC10.X2, J12.5
- net N$23: now also IC11.X6, JP3.2; no longer IC10.X1, J12.6
- net N$24: now also IC11.X4, JP3.1; no longer IC10.X0, J12.7
- net N$25: now also IC9.X2, JP1.8; no longer IC9.X5, J11.1
- net N$26: now also IC9.X1, JP1.7; no longer IC9.X4, J11.4
- net N$27: now also IC9.X0, JP1.6; no longer IC9.X3, J11.8
- net N$28: now also IC9.X3, JP1.5; no longer IC9.X7, J11.2
- net N$29: now also IC9.X5, JP1.4; no longer IC9.X6, J11.3
- net N$30: now also IC9.X7, JP1.3; no longer IC9.X2, J11.5
- net N$31: now also IC9.X6, JP1.2; no longer IC9.X1, J11.6
- net N$32: now also IC9.X4, JP1.1; no longer IC9.X0, J11.7
- net N$6: now also JP1.9, JP2.9, JP3.9; no longer J11.9, J12.9, J13.9
- net N$9: now also IC10.X0, JP2.6; no longer IC11.X7, J13.2
